File: sb-cnc-shield.kicad_pcb (KiCad board)
At the start: 2 copper layers, 68.6 x 53.3 mm, 63 parts, among them P1 XMOT, P2 YMOT, P3 ZMOT, P4 AMOT, P5 UART, P6 I2C, P7 ES_SETUP, P8 VMOT, SW1 RESET, U1 ARDUINO_UNO_SHIELD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

Commit message: upgraded to kicad 5
Changed lines of the file:
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@@
-(kicad_pcb (version 4) (host pcbnew 4.0.2-stable)
+(kicad_pcb (version 4) (host pcbnew 4.0.6)
   (general
     (links 174)
     (no_connects 0)
-    (area 94.030667 58.110001 189.306334 124.8608)
+    (area 94.105667 58.260001 189.231334 125.0132)
     (thickness 1.6)
-    (drawings 33)
+    (drawings 42)
     (tracks 788)
     (zones 0)
@@
     )
   )
+  (gr_text MS3 (at 159.8295 88.3285) (layer F.SilkS)
+    (effects (font (size 0.8 0.8) (thickness 0.125)))
+  )
+  (gr_text MS2 (at 159.8295 85.7885) (layer F.SilkS)
+    (effects (font (size 0.8 0.8) (thickness 0.125)))
+  )
+  (gr_text MS1 (at 159.893 83.2485) (layer F.SilkS)
+    (effects (font (size 0.8 0.8) (thickness 0.125)))
+  )
+  (gr_text MS3 (at 159.8295 108.6485) (layer F.SilkS)
+    (effects (font (size 0.8 0.8) (thickness 0.125)))
+  )
+  (gr_text MS2 (at 159.8295 106.1085) (layer F.SilkS)
+    (effects (font (size 0.8 0.8) (thickness 0.125)))
+  )
+  (gr_text MS1 (at 159.893 103.5685) (layer F.SilkS)
+    (effects (font (size 0.8 0.8) (thickness 0.125)))
+  )
+  (gr_text MS3 (at 137.7315 108.6485) (layer F.SilkS)
+    (effects (font (size 0.8 0.8) (thickness 0.125)))
+  )
+  (gr_text MS2 (at 137.7315 106.1085) (layer F.SilkS)
+    (effects (font (size 0.8 0.8) (thickness 0.125)))
+  )
+  (gr_text MS1 (at 137.795 103.5685) (layer F.SilkS)
+    (effects (font (size 0.8 0.8) (thickness 0.125)))
+  )
   (gr_text www.staticboards.com (at 139.573 117.221) (layer F.SilkS)
