File: sb-cnc-shield.sch (KiCad schematic (older format))
At the start: 62 parts, among them P1 XMOT, P2 YMOT, P3 ZMOT, P4 AMOT, P5 UART, P6 I2C, P7 ES_SETUP, P8 12V-36V, SW1 RESET, U1 ARDUINO_UNO_SHIELD, U2 X, U3 Y, U4 Z, U5 A

Commit message: upgraded to kicad 5
Parts:
- C1, C2, C3, C4: symbol CAP_ELECTRO-RESCUE-sb-cnc-shield -> sb-cnc-shield-rescue:CAP_ELECTRO-RESCUE-sb-cnc-shield
- JP1, JP10, JP11, JP12, JP13, JP14, JP15, JP16, JP17, JP18, JP19, JP2, JP20, JP21, JP22, JP23, JP24, JP25, JP26, JP27, JP28, JP29, JP3, JP30, JP31, JP32, JP33, JP34, JP35, JP36, JP37, JP38, JP39, JP4, JP5, JP6, JP7, JP8, JP9: symbol Jumper_NO_Small -> Device:Jumper_NO_Small
- P1, P2, P3, P4, P5, P6: symbol CONN_01X04 -> sb-cnc-shield-rescue:CONN_01X04
- P7: symbol CONN_01X03 -> sb-cnc-shield-rescue:CONN_01X03
- P8: symbol CONN_01X02 -> sb-cnc-shield-rescue:CONN_01X02
- R1, R2, R3, R4, R5: symbol R -> Device:R
- SW1: symbol SW_PUSH_4P -> sb-cnc-shield-rescue:SW_PUSH_4P
- U1: symbol ARDUINO_UNO_SHIELD -> sb-cnc-shield-rescue:ARDUINO_UNO_SHIELD
- U2, U3, U4, U5: symbol POLOLU_STEPPER_DRIVER -> sb-cnc-shield-rescue:POLOLU_STEPPER_DRIVER
